File: hardware/power.sch (KiCad schematic (older format))
At the start: 13 parts, among them Q36 Q_PMOS_GSD, U2 HT7333-1

Commit message: phase routet
Parts:
- removed C12: C, Capacitors_SMD:C_0603, symbol C
- removed C13: 100n, Capacitors_SMD:C_0603, symbol C
- removed C7: 1u, Capacitors_SMD:C_0603, symbol C
- added C23: 22u, Capacitors_SMD:C_0805, symbol C
- C19: renamed from C8; value C -> 22u; footprint Capacitors_SMD:C_0603 -> Capacitors_SMD:C_0805
- C21: renamed from C10; value C -> 22u; footprint Capacitors_SMD:C_0603 -> Capacitors_SMD:C_0805
- C22: renamed from C11; value C -> 22u; footprint Capacitors_SMD:C_0603 -> Capacitors_SMD:C_0805
- C24: renamed from C14; value 10u -> 22u
- Q36: value Q_PMOS_GSD -> AO3401
- renumbered C9 to C20
Connections:
- net GND: now also C23.1
- net Vjack: now also C23.2
Other:
- moved on the sheet: C24
Changed lines of the file:
@@
 P 3050 2150
 F 0 "Q36" H 3250 2200 50  0000 L CNN
-F 1 "Q_PMOS_GSD" H 3250 2100 50  0000 L CNN
+F 1 "AO3401" H 3250 2100 50  0000 L CNN
 F 2 "TO_SOT_Packages_SMD:SOT-23" H 3250 2250 50  0001 C CNN
 F 3 "" H 3050 2150 50  0001 C CNN
@@
 Connection ~ 3050 2700
 $Comp
-L C C7
-U 1 1 5AEC3E42
-P 3600 2350
-F 0 "C7" H 3625 2450 50  0000 L CNN
-F 1 "1u" H 3625 2250 50  0000 L CNN
-F 2 "Capacitors_SMD:C_0603" H 3638 2200 50  0001 C CNN
-F 3 "" H 3600 2350 50  0001 C CNN
-	1    3600 2350
-	1    0    0    -1
-$EndComp
-$Comp
-L C C9
+L C C20
 U 1 1 5AEC3E8F
 P 3900 2350
-F 0 "C9" H 3925 2450 50  0000 L CNN
+F 0 "C20" H 3925 2450 50  0000 L CNN
 F 1 "100n" H 3925 2250 50  0000 L CNN
 F 2 "Capacitors_SMD:C_0603" H 3938 2200 50  0001 C CNN
@@
 Connection ~ 3900 2050
 Wire Wire Line
-	3600 2200 3600 2050
-Connection ~ 3600 2050
-Wire Wire Line
 	2550 2500 2550 2600
 Wire Wire Line
 	2550 2600 5750 2600
 Wire Wire Line
-	3600 2500 3600 2700
+	3600 2600 3600 2700
 Connection ~ 2550 2500
 Wire Wire Line
@@
 Connection ~ 3900 2600
 $Comp
-L C C13
-U 1 1 5AEC3F5E
+L C C24
+U 1 1 5AEC4001
 P 4800 2350
-F 0 "C13" H 4825 2450 50  0000 L CNN
-F 1 "100n" H 4825 2250 50  0000 L CNN
+F 0 "C24" H 4825 2450 50  0000 L CNN
+F 1 "22u" H 4825 2250 50  0000 L CNN
 F 2 "Capacitors_SMD:C_0603" H 4838 2200 50  0001 C CNN
 F 3 "" H 4800 2350 50  0001 C CNN
@@
 	1    0    0    -1
 $EndComp
-$Comp
-L C C14
-U 1 1 5AEC4001
-P 5100 2350
-F 0 "C14" H 5125 2450 50  0000 L CNN
-F 1 "10u" H 5125 2250 50  0000 L CNN
-F 2 "Capacitors_SMD:C_0603" H 5138 2200 50  0001 C CNN
-F 3 "" H 5100 2350 50  0001 C CNN
-	1    5100 2350
-	1    0    0    -1
-$EndComp
 Wire Wire Line
-	5100 2600 5100 2500
+	4800 2600 4800 2500
 Connection ~ 4350 2600
-Wire Wire Line
-	4800 2500 4800 2600
-Connection ~ 4800 2600
-Wire Wire Line
-	4800 2200 4800 2050
 Wire Wire Line
 	4650 2050 6250 2050
 Wire Wire Line
-	5100 2050 5100 2200
+	4800 2050 4800 2200
 Connection ~ 4800 2050
-Connection ~ 5100 2050
 Wire Wire Line
 	3900 2050 3900 2200
 $Comp
-L C C8
+L C C19
 U 1 1 5AEC43A4
 P 3600 2850
-F 0 "C8" H 3625 2950 50  0000 L CNN
-F 1 "C" H 3625 2750 50  0000 L CNN
-F 2 "Capacitors_SMD:C_0603" H 3638 2700 50  0001 C CNN
+F 0 "C19" H 3625 2950 50  0000 L CNN
+F 1 "22u" H 3625 2750 50  0000 L CNN
+F 2 "Capacitors_SMD:C_0805" H 3638 2700 50  0001 C CNN
 F 3 "" H 3600 2850 50  0001 C CNN
 	1    3600 2850
@@
 $EndComp
 $Comp
-L C C10
+L C C21
 U 1 1 5AEC43CD
 P 3900 2850
-F 0 "C10" H 3925 2950 50  0000 L CNN
-F 1 "C" H 3925 2750 50  0000 L CNN
-F 2 "Capacitors_SMD:C_0603" H 3938 2700 50  0001 C CNN
+F 0 "C21" H 3925 2950 50  0000 L CNN
+F 1 "22u" H 3925 2750 50  0000 L CNN
+F 2 "Capacitors_SMD:C_0805" H 3938 2700 50  0001 C CNN
 F 3 "" H 3900 2850 50  0001 C CNN
 	1    3900 2850
@@
 $EndComp
 $Comp
-L C C11
+L C C22
 U 1 1 5AEC43FC
 P 4200 2850
-F 0 "C11" H 4225 2950 50  0000 L CNN
-F 1 "C" H 4225 2750 50  0000 L CNN
-F 2 "Capacitors_SMD:C_0603" H 4238 2700 50  0001 C CNN
+F 0 "C22" H 4225 2950 50  0000 L CNN
+F 1 "22u" H 4225 2750 50  0000 L CNN
+F 2 "Capacitors_SMD:C_0805" H 4238 2700 50  0001 C CNN
 F 3 "" H 4200 2850 50  0001 C CNN
 	1    4200 2850
-	1    0    0    -1
-$EndComp
-$Comp
-L C C12
-U 1 1 5AEC442D
-P 4500 2850
-F 0 "C12" H 4525 2950 50  0000 L CNN
-F 1 "C" H 4525 2750 50  0000 L CNN
-F 2 "Capacitors_SMD:C_0603" H 4538 2700 50  0001 C CNN
-F 3 "" H 4500 2850 50  0001 C CNN
-	1    4500 2850
 	1    0    0    -1
 $EndComp
@@
 	6150 3000 6150 3100
 Connection ~ 6150 3100
-Connection ~ 5100 2600
+Connection ~ 4800 2600
+$Comp
+L C C23
+U 1 1 5AE9BDFF
+P 4500 2850
+F 0 "C23" H 4525 2950 50  0000 L CNN
+F 1 "22u" H 4525 2750 50  0000 L CNN
+F 2 "Capacitors_SMD:C_0805" H 4538 2700 50  0001 C CNN
+F 3 "" H 4500 2850 50  0001 C CNN
+	1    4500 2850
+	1    0    0    -1
+$EndComp
 $EndSCHEMATC

Commit message: change to kicad 5
Parts:
- C19, C21, C22, C23: footprint Capacitors_SMD:C_0805 -> Capacitor_SMD:C_0805_2012Metric; symbol C -> Device:C
- C20, C24: footprint Capacitors_SMD:C_0603 -> Capacitor_SMD:C_0603_1608Metric; symbol C -> Device:C
- Q36: footprint TO_SOT_Packages_SMD:SOT-23 -> Package_TO_SOT_SMD:SOT-23; symbol Q_PMOS_GSD -> Device:Q_PMOS_GSD
- R41, R42, R43: footprint Resistors_SMD:R_0603 -> Resistor_SMD:R_0603_1608Metric; symbol R -> Device:R
- U2: footprint TO_SOT_Packages_SMD:SOT-89-3 -> Package_TO_SOT_SMD:SOT-89-3; symbol HT7333-1 -> Regulator_Linear:MCP1700-1202E_SOT89
Changed lines of the file:
@@
-EESchema Schematic File Version 2
-LIBS:74xgxx
-LIBS:74xx
-LIBS:ac-dc
-LIBS:actel
-LIBS:adc-dac
-LIBS:allegro
-LIBS:Altera
-LIBS:analog_devices
-LIBS:analog_switches
-LIBS:atmel
-LIBS:audio
-LIBS:battery_management
-LIBS:bbd
-LIBS:bosch
-LIBS:brooktre
-LIBS:cmos4000
-LIBS:cmos_ieee
-LIBS:conn
-LIBS:contrib
-LIBS:cypress
-LIBS:dc-dc
-LIBS:device
-LIBS:digital-audio
-LIBS:diode
-LIBS:display
-LIBS:dsp
-LIBS:elec-unifil
-LIBS:ESD_Protection
-LIBS:ftdi
-LIBS:gennum
-LIBS:graphic_symbols
-LIBS:hc11
-LIBS:infineon
-LIBS:intel
-LIBS:interface
-LIBS:intersil
-LIBS:ir
-LIBS:Lattice
-LIBS:leds
-LIBS:LEM
-LIBS:linear
-LIBS:logic_programmable
-LIBS:maxim
-LIBS:mechanical
-LIBS:memory
-LIBS:microchip
-LIBS:microchip_dspic33dsc
-LIBS:microchip_pic10mcu
-LIBS:microchip_pic12mcu
-LIBS:microchip_pic16mcu
-LIBS:microchip_pic18mcu
-LIBS:microchip_pic24mcu
-LIBS:microchip_pic32mcu
-LIBS:microcontrollers
-LIBS:modules
-LIBS:motor_drivers
-LIBS:motorola
-LIBS:motors
-LIBS:msp430
-LIBS:nordicsemi
-LIBS:nxp
-LIBS:nxp_armmcu
-LIBS:onsemi
-LIBS:opto
-LIBS:Oscillators
-LIBS:philips
-LIBS:power
-LIBS:powerint
-LIBS:Power_Management
-LIBS:pspice
-LIBS:references
-LIBS:regul
-LIBS:relays
-LIBS:rfcom
-LIBS:RFSolutions
-LIBS:sensors
-LIBS:silabs
-LIBS:siliconi
-LIBS:stm8
-LIBS:stm32
-LIBS:supertex
-LIBS:switches
-LIBS:texas
-LIBS:transf
-LIBS:transistors
-LIBS:triac_thyristor
-LIBS:ttl_ieee
-LIBS:valves
-LIBS:video
-LIBS:wiznet
-LIBS:Worldsemi
-LIBS:Xicor
-LIBS:xilinx
-LIBS:zetex
-LIBS:Zilog
-LIBS:gmcontrol
+EESchema Schematic File Version 4
 LIBS:gmcontrol-cache
-EELAYER 25 0
+EELAYER 26 0
 EELAYER END
 $Descr A4 11693 8268
@@
 Vmotor
 $Comp
-L HT7333-1 U2
+L Regulator_Linear:MCP1700-1202E_SOT89 U2
 U 1 1 5AEC37F4
 P 4350 2050
+AR Path="/5AEC37F4" Ref="U2"  Part="1"
+AR Path="/5AEC260A/5AEC37F4" Ref="U2"  Part="1"
 F 0 "U2" H 4200 2175 50  0000 C CNN
 F 1 "HT7333-1" H 4350 2175 50  0000 L CNN
-F 2 "TO_SOT_Packages_SMD:SOT-89-3" H 4350 2300 50  0001 C CIN
+F 2 "Package_TO_SOT_SMD:SOT-89-3" H 4350 2300 50  0001 C CIN
 F 3 "" H 4350 2050 50  0001 C CNN
 	1    4350 2050
@@
 $EndComp
 $Comp
-L Q_PMOS_GSD Q36
+L Device:Q_PMOS_GSD Q36
 U 1 1 5AEC3823
 P 3050 2150
+AR Path="/5AEC3823" Ref="Q36"  Part="1"
+AR Path="/5AEC260A/5AEC3823" Ref="Q36"  Part="1"
 F 0 "Q36" H 3250 2200 50  0000 L CNN
 F 1 "AO3401" H 3250 2100 50  0000 L CNN
-F 2 "TO_SOT_Packages_SMD:SOT-23" H 3250 2250 50  0001 C CNN
+F 2 "Package_TO_SOT_SMD:SOT-23" H 3250 2250 50  0001 C CNN
 F 3 "" H 3050 2150 50  0001 C CNN
 	1    3050 2150
@@
 $EndComp
 $Comp
-L R R41
+L Device:R R41
 U 1 1 5AEC38AD
 P 2750 2500
+AR Path="/5AEC38AD" Ref="R41"  Part="1"
+AR Path="/5AEC260A/5AEC38AD" Ref="R41"  Part="1"
 F 0 "R41" V 2830 2500 50  0000 C CNN
 F 1 "10k" V 2750 2500 50  0000 C CNN
-F 2 "Resistors_SMD:R_0603" V 2680 2500 50  0001 C CNN
+F 2 "Resistor_SMD:R_0603_1608Metric" V 2680 2500 50  0001 C CNN
 F 3 "" H 2750 2500 50  0001 C CNN
 	1    2750 2500
@@
 	2850 2050 2200 2050
 Wire Wire Line
-	3250 2050 4050 2050
-Wire Wire Line
-	2200 2500 2600 2500
-Wire Wire Line
-	3050 2350 3050 2700
+	3250 2050 3400 2050
+Wire Wire Line
+	2200 2500 2550 2500
+Wire Wire Line
+	3050 2350 3050 2500
 Wire Wire Line
 	3050 2500 2900 2500
 Wire Wire Line
-	2200 2700 3400 2700
+	2200 2700 3050 2700
 Connection ~ 3050 2500
 Wire Wire Line
-	3400 2050 3400 3100
+	3400 2050 3400 2700
 Connection ~ 3050 2700
 $Comp
-L C C20
+L Device:C C20
 U 1 1 5AEC3E8F
 P 3900 2350
+AR Path="/5AEC3E8F" Ref="C20"  Part="1"
+AR Path="/5AEC260A/5AEC3E8F" Ref="C20"  Part="1"
 F 0 "C20" H 3925 2450 50  0000 L CNN
 F 1 "100n" H 3925 2250 50  0000 L CNN
-F 2 "Capacitors_SMD:C_0603" H 3938 2200 50  0001 C CNN
+F 2 "Capacitor_SMD:C_0603_1608Metric" H 3938 2200 50  0001 C CNN
 F 3 "" H 3900 2350 50  0001 C CNN
 	1    3900 2350
@@
 	2550 2500 2550 2600
 Wire Wire Line
-	2550 2600 5750 2600
+	2550 2600 3600 2600
 Wire Wire Line
 	3600 2600 3600 2700
 Connection ~ 2550 2500
 Wire Wire Line
-	3900 2500 3900 2700
+	3900 2500 3900 2600
 Connection ~ 3600 2600
 Wire Wire Line
@@
 Connection ~ 3900 2600
 $Comp
-L C C24
+L Device:C C24
 U 1 1 5AEC4001
 P 4800 2350
+AR Path="/5AEC4001" Ref="C24"  Part="1"
+AR Path="/5AEC260A/5AEC4001" Ref="C24"  Part="1"
 F 0 "C24" H 4825 2450 50  0000 L CNN
 F 1 "22u" H 4825 2250 50  0000 L CNN
-F 2 "Capacitors_SMD:C_0603" H 4838 2200 50  0001 C CNN
+F 2 "Capacitor_SMD:C_0603_1608Metric" H 4838 2200 50  0001 C CNN
 F 3 "" H 4800 2350 50  0001 C CNN
 	1    4800 2350
@@
 Connection ~ 4350 2600
 Wire Wire Line
-	4650 2050 6250 2050
+	4650 2050 4800 2050
 Wire Wire Line
 	4800 2050 4800 2200
@@
 	3900 2050 3900 2200
 $Comp
-L C C19
+L Device:C C19
 U 1 1 5AEC43A4
 P 3600 2850
+AR Path="/5AEC43A4" Ref="C19"  Part="1"
+AR Path="/5AEC260A/5AEC43A4" Ref="C19"  Part="1"
 F 0 "C19" H 3625 2950 50  0000 L CNN
 F 1 "22u" H 3625 2750 50  0000 L CNN
-F 2 "Capacitors_SMD:C_0805" H 3638 2700 50  0001 C CNN
+F 2 "Capacitor_SMD:C_0805_2012Metric" H 3638 2700 50  0001 C CNN
 F 3 "" H 3600 2850 50  0001 C CNN
 	1    3600 2850
@@
 $EndComp
 $Comp
-L C C21
+L Device:C C21
 U 1 1 5AEC43CD
 P 3900 2850
+AR Path="/5AEC43CD" Ref="C21"  Part="1"
+AR Path="/5AEC260A/5AEC43CD" Ref="C21"  Part="1"
 F 0 "C21" H 3925 2950 50  0000 L CNN
 F 1 "22u" H 3925 2750 50  0000 L CNN
-F 2 "Capacitors_SMD:C_0805" H 3938 2700 50  0001 C CNN
+F 2 "Capacitor_SMD:C_0805_2012Metric" H 3938 2700 50  0001 C CNN
 F 3 "" H 3900 2850 50  0001 C CNN
 	1    3900 2850
@@
 $EndComp
 $Comp
-L C C22
+L Device:C C22
 U 1 1 5AEC43FC
 P 4200 2850
+AR Path="/5AEC43FC" Ref="C22"  Part="1"
+AR Path="/5AEC260A/5AEC43FC" Ref="C22"  Part="1"
 F 0 "C22" H 4225 2950 50  0000 L CNN
 F 1 "22u" H 4225 2750 50  0000 L CNN
-F 2 "Capacitors_SMD:C_0805" H 4238 2700 50  0001 C CNN
+F 2 "Capacitor_SMD:C_0805_2012Metric" H 4238 2700 50  0001 C CNN
 F 3 "" H 4200 2850 50  0001 C CNN
 	1    4200 2850
@@
 $EndComp
 Wire Wire Line
-	3400 3100 6250 3100
+	3400 3100 3600 3100
 Wire Wire Line
 	4500 3100 4500 3000
@@
 SENSE_Vmotor
 $Comp
-L R R42
+L Device:R R42
 U 1 1 5AEC4801
 P 5900 2600
+AR Path="/5AEC4801" Ref="R42"  Part="1"
+AR Path="/5AEC260A/5AEC4801" Ref="R42"  Part="1"
 F 0 "R42" V 5980 2600 50  0000 C CNN
 F 1 "10k" V 5900 2600 50  0000 C CNN
-F 2 "Resistors_SMD:R_0603" V 5830 2600 50  0001 C CNN
+F 2 "Resistor_SMD:R_0603_1608Metric" V 5830 2600 50  0001 C CNN
 F 3 "" H 5900 2600 50  0001 C CNN
 	1    5900 2600
@@
 $EndComp
 $Comp
-L R R43
+L Device:R R43
 U 1 1 5AEC4917
 P 6150 2850
+AR Path="/5AEC4917" Ref="R43"  Part="1"
+AR Path="/5AEC260A/5AEC4917" Ref="R43"  Part="1"
 F 0 "R43" V 6230 2850 50  0000 C CNN
 F 1 "1k" V 6150 2850 50  0000 C CNN
-F 2 "Resistors_SMD:R_0603" V 6080 2850 50  0001 C CNN
+F 2 "Resistor_SMD:R_0603_1608Metric" V 6080 2850 50  0001 C CNN
 F 3 "" H 6150 2850 50  0001 C CNN
 	1    6150 2850
@@
 	6150 2700 6150 2600
 Wire Wire Line
-	6050 2600 6250 2600
+	6050 2600 6150 2600
 Connection ~ 6150 2600
 Wire Wire Line
@@
 Connection ~ 4800 2600
 $Comp
-L C C23
+L Device:C C23
 U 1 1 5AE9BDFF
 P 4500 2850
+AR Path="/5AE9BDFF" Ref="C23"  Part="1"
+AR Path="/5AEC260A/5AE9BDFF" Ref="C23"  Part="1"
 F 0 "C23" H 4525 2950 50  0000 L CNN
 F 1 "22u" H 4525 2750 50  0000 L CNN
-F 2 "Capacitors_SMD:C_0805" H 4538 2700 50  0001 C CNN
+F 2 "Capacitor_SMD:C_0805_2012Metric" H 4538 2700 50  0001 C CNN
 F 3 "" H 4500 2850 50  0001 C CNN
 	1    4500 2850
 	1    0    0    -1
 $EndComp
+Wire Wire Line
+	3050 2500 3050 2700
+Wire Wire Line
+	3050 2700 3400 2700
+Wire Wire Line
+	3400 2050 3900 2050
+Wire Wire Line
+	3900 2050 4050 2050
+Wire Wire Line
+	2550 2500 2600 2500
+Wire Wire Line
+	3600 2600 3900 2600
+Wire Wire Line
+	3900 2600 3900 2700
+Wire Wire Line
+	3900 2600 4200 2600
+Wire Wire Line
+	4350 2600 4500 2600
+Wire Wire Line
+	4800 2050 6250 2050
+Wire Wire Line
+	3400 2700 3400 3100
+Wire Wire Line
+	4200 3100 4500 3100
+Wire Wire Line
+	3900 3100 4200 3100
+Wire Wire Line
+	3600 3100 3900 3100
+Wire Wire Line
+	4200 2600 4350 2600
+Wire Wire Line
+	4500 2600 4800 2600
+Wire Wire Line
+	4500 3100 6150 3100
+Wire Wire Line
+	6150 2600 6250 2600
+Wire Wire Line
+	6150 3100 6250 3100
+Wire Wire Line
+	4800 2600 5750 2600
 $EndSCHEMATC

Commit message: smaller footprints
Parts:
- C19, C21, C22, C23: footprint Capacitor_SMD:C_0805_2012Metric -> _Generic:0805_Small
- C20, C24: footprint Capacitor_SMD:C_0603_1608Metric -> _Generic:0603_Small
- Q36: footprint Package_TO_SOT_SMD:SOT-23 -> _Generic:SOT-23_Small
- R41, R42, R43: footprint Resistor_SMD:R_0603_1608Metric -> _Generic:0603_Small
Changed lines of the file:
@@
 F 0 "Q36" H 3250 2200 50  0000 L CNN
 F 1 "AO3401" H 3250 2100 50  0000 L CNN
-F 2 "Package_TO_SOT_SMD:SOT-23" H 3250 2250 50  0001 C CNN
+F 2 "_Generic:SOT-23_Small" H 3250 2250 50  0001 C CNN
 F 3 "" H 3050 2150 50  0001 C CNN
 	1    3050 2150
@@
 F 0 "R41" V 2830 2500 50  0000 C CNN
 F 1 "10k" V 2750 2500 50  0000 C CNN
-F 2 "Resistor_SMD:R_0603_1608Metric" V 2680 2500 50  0001 C CNN
+F 2 "_Generic:0603_Small" V 2680 2500 50  0001 C CNN
 F 3 "" H 2750 2500 50  0001 C CNN
 	1    2750 2500
@@
 F 0 "C20" H 3925 2450 50  0000 L CNN
 F 1 "100n" H 3925 2250 50  0000 L CNN
-F 2 "Capacitor_SMD:C_0603_1608Metric" H 3938 2200 50  0001 C CNN
+F 2 "_Generic:0603_Small" H 3938 2200 50  0001 C CNN
 F 3 "" H 3900 2350 50  0001 C CNN
 	1    3900 2350
@@
 F 0 "C24" H 4825 2450 50  0000 L CNN
 F 1 "22u" H 4825 2250 50  0000 L CNN
-F 2 "Capacitor_SMD:C_0603_1608Metric" H 4838 2200 50  0001 C CNN
+F 2 "_Generic:0603_Small" H 4838 2200 50  0001 C CNN
 F 3 "" H 4800 2350 50  0001 C CNN
 	1    4800 2350
@@
 F 0 "C19" H 3625 2950 50  0000 L CNN
 F 1 "22u" H 3625 2750 50  0000 L CNN
-F 2 "Capacitor_SMD:C_0805_2012Metric" H 3638 2700 50  0001 C CNN
+F 2 "_Generic:0805_Small" H 3638 2700 50  0001 C CNN
 F 3 "" H 3600 2850 50  0001 C CNN
 	1    3600 2850
@@
 F 0 "C21" H 3925 2950 50  0000 L CNN
 F 1 "22u" H 3925 2750 50  0000 L CNN
-F 2 "Capacitor_SMD:C_0805_2012Metric" H 3938 2700 50  0001 C CNN
+F 2 "_Generic:0805_Small" H 3938 2700 50  0001 C CNN
 F 3 "" H 3900 2850 50  0001 C CNN
 	1    3900 2850
@@
 F 0 "C22" H 4225 2950 50  0000 L CNN
 F 1 "22u" H 4225 2750 50  0000 L CNN
-F 2 "Capacitor_SMD:C_0805_2012Metric" H 4238 2700 50  0001 C CNN
+F 2 "_Generic:0805_Small" H 4238 2700 50  0001 C CNN
 F 3 "" H 4200 2850 50  0001 C CNN
 	1    4200 2850
@@
 F 0 "R42" V 5980 2600 50  0000 C CNN
 F 1 "10k" V 5900 2600 50  0000 C CNN
-F 2 "Resistor_SMD:R_0603_1608Metric" V 5830 2600 50  0001 C CNN
+F 2 "_Generic:0603_Small" V 5830 2600 50  0001 C CNN
 F 3 "" H 5900 2600 50  0001 C CNN
 	1    5900 2600
@@
 F 0 "R43" V 6230 2850 50  0000 C CNN
 F 1 "1k" V 6150 2850 50  0000 C CNN
-F 2 "Resistor_SMD:R_0603_1608Metric" V 6080 2850 50  0001 C CNN
+F 2 "_Generic:0603_Small" V 6080 2850 50  0001 C CNN
 F 3 "" H 6150 2850 50  0001 C CNN
 	1    6150 2850
@@
 F 0 "C23" H 4525 2950 50  0000 L CNN
 F 1 "22u" H 4525 2750 50  0000 L CNN
-F 2 "Capacitor_SMD:C_0805_2012Metric" H 4538 2700 50  0001 C CNN
+F 2 "_Generic:0805_Small" H 4538 2700 50  0001 C CNN
 F 3 "" H 4500 2850 50  0001 C CNN
 	1    4500 2850

Commit message: power layout
Parts:
- added C25, C26, C27, C28: 22u, _Generic:0805_Small, symbol Device:C
Connections:
- net GND: now also C25.1, C26.1, C27.1, C28.1
- net Vjack: now also C25.2, C26.2, C27.2, C28.2
Changed lines of the file:
@@
 	4500 2600 4800 2600
 Wire Wire Line
-	4500 3100 6150 3100
+	4500 3100 4800 3100
 Wire Wire Line
 	6150 2600 6250 2600
@@
 	6150 3100 6250 3100
 Wire Wire Line
-	4800 2600 5750 2600
+	4800 2600 5100 2600
+$Comp
+L Device:C C25
+U 1 1 5AEDFCAE
+P 4800 2850
+F 0 "C25" H 4825 2950 50  0000 L CNN
+F 1 "22u" H 4825 2750 50  0000 L CNN
+F 2 "_Generic:0805_Small" H 4838 2700 50  0001 C CNN
+F 3 "" H 4800 2850 50  0001 C CNN
+	1    4800 2850
+	1    0    0    -1
+$EndComp
+$Comp
+L Device:C C26
+U 1 1 5AEDFCFC
+P 5100 2850
+F 0 "C26" H 5125 2950 50  0000 L CNN
+F 1 "22u" H 5125 2750 50  0000 L CNN
+F 2 "_Generic:0805_Small" H 5138 2700 50  0001 C CNN
+F 3 "" H 5100 2850 50  0001 C CNN
+	1    5100 2850
+	1    0    0    -1
+$EndComp
+$Comp
+L Device:C C27
+U 1 1 5AEDFD83
+P 5400 2850
+F 0 "C27" H 5425 2950 50  0000 L CNN
+F 1 "22u" H 5425 2750 50  0000 L CNN
+F 2 "_Generic:0805_Small" H 5438 2700 50  0001 C CNN
+F 3 "" H 5400 2850 50  0001 C CNN
+	1    5400 2850
+	1    0    0    -1
+$EndComp
+$Comp
+L Device:C C28
+U 1 1 5AEDFDC3
+P 5700 2850
+F 0 "C28" H 5725 2950 50  0000 L CNN
+F 1 "22u" H 5725 2750 50  0000 L CNN
+F 2 "_Generic:0805_Small" H 5738 2700 50  0001 C CNN
+F 3 "" H 5700 2850 50  0001 C CNN
+	1    5700 2850
+	1    0    0    -1
+$EndComp
+Wire Wire Line
+	4800 2700 4800 2600
+Wire Wire Line
+	5100 2700 5100 2600
+Connection ~ 5100 2600
+Wire Wire Line
+	5100 2600 5400 2600
+Wire Wire Line
+	5400 2700 5400 2600
+Connection ~ 5400 2600
+Wire Wire Line
+	5400 2600 5700 2600
+Wire Wire Line
+	5700 2700 5700 2600
+Connection ~ 5700 2600
+Wire Wire Line
+	5700 2600 5750 2600
+Wire Wire Line
+	5700 3000 5700 3100
+Connection ~ 5700 3100
+Wire Wire Line
+	5700 3100 6150 3100
+Wire Wire Line
+	5400 3000 5400 3100
+Connection ~ 5400 3100
+Wire Wire Line
+	5400 3100 5700 3100
+Wire Wire Line
+	5100 3000 5100 3100
+Connection ~ 5100 3100
+Wire Wire Line
+	5100 3100 5400 3100
+Wire Wire Line
+	4800 3000 4800 3100
+Connection ~ 4800 3100
+Wire Wire Line
+	4800 3100 5100 3100
 $EndSCHEMATC

Commit message: basic layout
Parts:
- added C29, C30: 22u, _Generic:0805_Small, symbol Device:C
Connections:
- net GND: now also C29.1, C30.1
- net Vjack: now also C29.2, C30.2
Other:
- moved on the sheet: R42, R43
Changed lines of the file:
@@
 Text HLabel 6250 2050 2    60   Output ~ 0
 3.3V
-Text HLabel 6250 3100 2    60   Output ~ 0
+Text HLabel 6950 3100 2    60   Output ~ 0
 Vmotor
 $Comp
@@
 Connection ~ 4500 2600
 Connection ~ 4500 3100
-Text HLabel 6250 2600 2    60   Output ~ 0
+Text HLabel 6950 2600 2    60   Output ~ 0
 SENSE_Vmotor
 $Comp
 L Device:R R42
 U 1 1 5AEC4801
-P 5900 2600
-F 0 "R42" V 5980 2600 50  0000 C CNN
-F 1 "10k" V 5900 2600 50  0000 C CNN
-F 2 "_Generic:0603_Small" V 5830 2600 50  0001 C CNN
-F 3 "" H 5900 2600 50  0001 C CNN
-	1    5900 2600
+P 6600 2600
+F 0 "R42" V 6680 2600 50  0000 C CNN
+F 1 "10k" V 6600 2600 50  0000 C CNN
+F 2 "_Generic:0603_Small" V 6530 2600 50  0001 C CNN
+F 3 "" H 6600 2600 50  0001 C CNN
+	1    6600 2600
 	0    1    1    0
 $EndComp
@@
 L Device:R R43
 U 1 1 5AEC4917
-P 6150 2850
-F 0 "R43" V 6230 2850 50  0000 C CNN
-F 1 "1k" V 6150 2850 50  0000 C CNN
-F 2 "_Generic:0603_Small" V 6080 2850 50  0001 C CNN
-F 3 "" H 6150 2850 50  0001 C CNN
-	1    6150 2850
-	1    0    0    -1
-$EndComp
-Wire Wire Line
-	6150 2700 6150 2600
-Wire Wire Line
-	6050 2600 6150 2600
-Connection ~ 6150 2600
-Wire Wire Line
-	6150 3000 6150 3100
-Connection ~ 6150 3100
+P 6850 2850
+F 0 "R43" V 6930 2850 50  0000 C CNN
+F 1 "1k" V 6850 2850 50  0000 C CNN
+F 2 "_Generic:0603_Small" V 6780 2850 50  0001 C CNN
+F 3 "" H 6850 2850 50  0001 C CNN
+	1    6850 2850
+	1    0    0    -1
+$EndComp
+Wire Wire Line
+	6850 2700 6850 2600
+Wire Wire Line
+	6750 2600 6850 2600
+Connection ~ 6850 2600
+Wire Wire Line
+	6850 3000 6850 3100
+Connection ~ 6850 3100
 Connection ~ 4800 2600
 $Comp
@@
 	4500 3100 4800 3100
 Wire Wire Line
-	6150 2600 6250 2600
-Wire Wire Line
-	6150 3100 6250 3100
+	6850 2600 6950 2600
+Wire Wire Line
+	6850 3100 6950 3100
 Wire Wire Line
 	4800 2600 5100 2600
@@
 Connection ~ 5700 2600
 Wire Wire Line
-	5700 2600 5750 2600
+	5700 2600 6000 2600
 Wire Wire Line
 	5700 3000 5700 3100
 Connection ~ 5700 3100
 Wire Wire Line
-	5700 3100 6150 3100
+	5700 3100 6000 3100
 Wire Wire Line
 	5400 3000 5400 3100
@@
 Wire Wire Line
 	4800 3100 5100 3100
+$Comp
+L Device:C C29
+U 1 1 5AEE2F7A
+P 6000 2850
+F 0 "C29" H 6025 2950 50  0000 L CNN
+F 1 "22u" H 6025 2750 50  0000 L CNN
+F 2 "_Generic:0805_Small" H 6038 2700 50  0001 C CNN
+F 3 "" H 6000 2850 50  0001 C CNN
+	1    6000 2850
+	1    0    0    -1
+$EndComp
+$Comp
+L Device:C C30
+U 1 1 5AEE2FE2
+P 6300 2850
+F 0 "C30" H 6325 2950 50  0000 L CNN
+F 1 "22u" H 6325 2750 50  0000 L CNN
+F 2 "_Generic:0805_Small" H 6338 2700 50  0001 C CNN
+F 3 "" H 6300 2850 50  0001 C CNN
+	1    6300 2850
+	1    0    0    -1
+$EndComp
+Wire Wire Line
+	6000 3000 6000 3100
+Connection ~ 6000 3100
+Wire Wire Line
+	6000 3100 6300 3100
+Wire Wire Line
+	6000 2700 6000 2600
+Connection ~ 6000 2600
+Wire Wire Line
+	6000 2600 6300 2600
+Wire Wire Line
+	6300 2700 6300 2600
+Connection ~ 6300 2600
+Wire Wire Line
+	6300 2600 6450 2600
+Wire Wire Line
+	6300 3000 6300 3100
+Connection ~ 6300 3100
+Wire Wire Line
+	6300 3100 6850 3100
 $EndSCHEMATC
