File: hardware/phase_driver.sch (KiCad schematic (older format))
At the start: 15 parts

Commit message: power, mcu
Parts:
- Q7, Q8: renamed from Q?; footprint (none) -> TO_SOT_Packages_SMD:PQFN_8x8
- R1, R2, R3, R4, R5, R6, R7: renamed from R?; footprint (none) -> Resistors_SMD:R_0603
- gave numbers to parts that had none: 6
Connections:
- net HIN renamed PHASE_H
- net LIN renamed PHASE_L
- net Phase renamed PHASE
- net Sense renamed SENSE
- net VGateH renamed Vgh
- net VGateL renamed Vgl
- net VMotor renamed Vmotor

Commit message: phase routet
Parts:
- added C1, C2: 1u, Capacitors_SMD:C_0603, symbol C
- Q7, Q8: value Q_NMOS_SGD -> AON7212; footprint TO_SOT_Packages_SMD:PQFN_8x8 -> gmcontrol:DFN3x3A_8L_EP1_P
Connections:
- net GND: now also C1.2, C2.2
- net Vgh: now also C2.1
- net Vgl: now also C1.1
Changed lines of the file:
@@
 $Descr A4 11693 8268
 encoding utf-8
-Sheet 4 8
+Sheet 2 8
 Title ""
 Date ""
@@
 AR Path="/5AEA2A43/5AE6CAAE" Ref="Q21"  Part="1"
 AR Path="/5AEA319E/5AE6CAAE" Ref="Q29"  Part="1"
-F 0 "Q13" H 7300 3825 50  0000 L CNN
+F 0 "Q5" H 7300 3825 50  0000 L CNN
 F 1 "BC817" H 7300 3750 50  0000 L CNN
 F 2 "TO_SOT_Packages_SMD:SOT-23" H 7300 3675 50  0001 L CIN
@@
 AR Path="/5AEA2A43/5AE6CB43" Ref="Q18"  Part="1"
 AR Path="/5AEA319E/5AE6CB43" Ref="Q26"  Part="1"
-F 0 "Q10" H 6550 4425 50  0000 L CNN
+F 0 "Q2" H 6550 4425 50  0000 L CNN
 F 1 "BC817" H 6550 4350 50  0000 L CNN
 F 2 "TO_SOT_Packages_SMD:SOT-23" H 6550 4275 50  0001 L CIN
@@
 AR Path="/5AEA2A43/5AE6CB8C" Ref="Q22"  Part="1"
 AR Path="/5AEA319E/5AE6CB8C" Ref="Q30"  Part="1"
-F 0 "Q14" H 7300 4425 50  0000 L CNN
+F 0 "Q6" H 7300 4425 50  0000 L CNN
 F 1 "BC807" H 7300 4350 50  0000 L CNN
 F 2 "TO_SOT_Packages_SMD:SOT-23" H 7300 4275 50  0001 L CIN
@@
 AR Path="/5AEA2A43/5AE6CC83" Ref="R22"  Part="1"
 AR Path="/5AEA319E/5AE6CC83" Ref="R29"  Part="1"
-F 0 "R15" V 6530 3800 50  0000 C CNN
+F 0 "R5" V 6530 3800 50  0000 C CNN
 F 1 "470" V 6450 3800 50  0000 C CNN
 F 2 "Resistors_SMD:R_0603" V 6380 3800 50  0001 C CNN
@@
 AR Path="/5AEA2A43/5AE6CCF2" Ref="R19"  Part="1"
 AR Path="/5AEA319E/5AE6CCF2" Ref="R26"  Part="1"
-F 0 "R12" V 5880 4350 50  0000 C CNN
+F 0 "R2" V 5880 4350 50  0000 C CNN
 F 1 "470" V 5800 4350 50  0000 C CNN
 F 2 "Resistors_SMD:R_0603" V 5730 4350 50  0001 C CNN
@@
 AR Path="/5AEA2A43/5AE6CEBE" Ref="Q24"  Part="1"
 AR Path="/5AEA319E/5AE6CEBE" Ref="Q32"  Part="1"
-F 0 "Q16" H 7950 4100 50  0000 L CNN
-F 1 "Q_NMOS_SGD" H 7950 4000 50  0000 L CNN
-F 2 "TO_SOT_Packages_SMD:PQFN_8x8" H 7950 4150 50  0001 C CNN
+F 0 "Q8" H 7950 4100 50  0000 L CNN
+F 1 "AON7212" H 7950 4000 50  0000 L CNN
+F 2 "gmcontrol:DFN3x3A_8L_EP1_P" H 7950 4150 50  0001 C CNN
 F 3 "" H 7750 4050 50  0001 C CNN
 	1    7750 4050
@@
 AR Path="/5AEA2A43/5AE6DEA8" Ref="Q19"  Part="1"
 AR Path="/5AEA319E/5AE6DEA8" Ref="Q27"  Part="1"
-F 0 "Q11" H 7300 1625 50  0000 L CNN
+F 0 "Q3" H 7300 1625 50  0000 L CNN
 F 1 "BC817" H 7300 1550 50  0000 L CNN
 F 2 "TO_SOT_Packages_SMD:SOT-23" H 7300 1475 50  0001 L CIN
@@
 AR Path="/5AEA2A43/5AE6DEAF" Ref="Q17"  Part="1"
 AR Path="/5AEA319E/5AE6DEAF" Ref="Q25"  Part="1"
-F 0 "Q9" H 6550 2225 50  0000 L CNN
+F 0 "Q1" H 6550 2225 50  0000 L CNN
 F 1 "BC817" H 6550 2150 50  0000 L CNN
 F 2 "TO_SOT_Packages_SMD:SOT-23" H 6550 2075 50  0001 L CIN
@@
 AR Path="/5AEA2A43/5AE6DEB6" Ref="Q20"  Part="1"
 AR Path="/5AEA319E/5AE6DEB6" Ref="Q28"  Part="1"
-F 0 "Q12" H 7300 2225 50  0000 L CNN
+F 0 "Q4" H 7300 2225 50  0000 L CNN
 F 1 "BC807" H 7300 2150 50  0000 L CNN
 F 2 "TO_SOT_Packages_SMD:SOT-23" H 7300 2075 50  0001 L CIN
@@
 AR Path="/5AEA2A43/5AE6DEBD" Ref="R20"  Part="1"
 AR Path="/5AEA319E/5AE6DEBD" Ref="R27"  Part="1"
-F 0 "R13" V 6530 1600 50  0000 C CNN
+F 0 "R3" V 6530 1600 50  0000 C CNN
 F 1 "470" V 6450 1600 50  0000 C CNN
 F 2 "Resistors_SMD:R_0603" V 6380 1600 50  0001 C CNN
@@
 AR Path="/5AEA2A43/5AE6DEC4" Ref="R18"  Part="1"
 AR Path="/5AEA319E/5AE6DEC4" Ref="R25"  Part="1"
-F 0 "R11" V 5880 2150 50  0000 C CNN
+F 0 "R1" V 5880 2150 50  0000 C CNN
 F 1 "470" V 5800 2150 50  0000 C CNN
 F 2 "Resistors_SMD:R_0603" V 5730 2150 50  0001 C CNN
@@
 AR Path="/5AEA2A43/5AE6DEDD" Ref="Q23"  Part="1"
 AR Path="/5AEA319E/5AE6DEDD" Ref="Q31"  Part="1"
-F 0 "Q15" H 7950 1900 50  0000 L CNN
-F 1 "Q_NMOS_SGD" H 7950 1800 50  0000 L CNN
-F 2 "TO_SOT_Packages_SMD:PQFN_8x8" H 7950 1950 50  0001 C CNN
+F 0 "Q7" H 7950 1900 50  0000 L CNN
+F 1 "AON7212" H 7950 1800 50  0000 L CNN
+F 2 "gmcontrol:DFN3x3A_8L_EP1_P" H 7950 1950 50  0001 C CNN
 F 3 "" H 7750 1850 50  0001 C CNN
 	1    7750 1850
@@
 AR Path="/5AEA2A43/5AE6E0AE" Ref="R21"  Part="1"
 AR Path="/5AEA319E/5AE6E0AE" Ref="R28"  Part="1"
-F 0 "R14" V 6530 2700 50  0000 C CNN
+F 0 "R4" V 6530 2700 50  0000 C CNN
 F 1 "100" V 6450 2700 50  0000 C CNN
 F 2 "Resistors_SMD:R_0603" V 6380 2700 50  0001 C CNN
@@
 AR Path="/5AEA2A43/5AE87A58" Ref="R23"  Part="1"
 AR Path="/5AEA319E/5AE87A58" Ref="R30"  Part="1"
-F 0 "R16" V 8830 3450 50  0000 C CNN
+F 0 "R6" V 8830 3450 50  0000 C CNN
 F 1 "10k" V 8750 3450 50  0000 C CNN
 F 2 "Resistors_SMD:R_0603" V 8680 3450 50  0001 C CNN
@@
 AR Path="/5AEA2A43/5AE87B6A" Ref="R24"  Part="1"
 AR Path="/5AEA319E/5AE87B6A" Ref="R31"  Part="1"
-F 0 "R17" V 8830 3950 50  0000 C CNN
+F 0 "R7" V 8830 3950 50  0000 C CNN
 F 1 "1k" V 8750 3950 50  0000 C CNN
 F 2 "Resistors_SMD:R_0603" V 8680 3950 50  0001 C CNN
@@
 Wire Wire Line
 	7200 2950 7200 2350
+$Comp
+L C C1
+U 1 1 5AE9E83C
+P 6050 3800
+AR Path="/5AE5B5EB/5AE9E83C" Ref="C1"  Part="1"
+AR Path="/5AEA1DF0/5AE9E83C" Ref="C11"  Part="1"
+AR Path="/5AEA2A43/5AE9E83C" Ref="C13"  Part="1"
+AR Path="/5AEA319E/5AE9E83C" Ref="C15"  Part="1"
+F 0 "C1" H 6075 3900 50  0000 L CNN
+F 1 "1u" H 6075 3700 50  0000 L CNN
+F 2 "Capacitors_SMD:C_0603" H 6088 3650 50  0001 C CNN
+F 3 "" H 6050 3800 50  0001 C CNN
+	1    6050 3800
+	1    0    0    -1
+$EndComp
+Wire Wire Line
+	6050 3650 6050 3450
+Connection ~ 6050 3450
+Wire Wire Line
+	6050 3950 6050 4700
+Connection ~ 6050 4700
+$Comp
+L C C2
+U 1 1 5AE9EAA8
+P 6100 1600
+AR Path="/5AE5B5EB/5AE9EAA8" Ref="C2"  Part="1"
+AR Path="/5AEA1DF0/5AE9EAA8" Ref="C12"  Part="1"
+AR Path="/5AEA2A43/5AE9EAA8" Ref="C14"  Part="1"
+AR Path="/5AEA319E/5AE9EAA8" Ref="C16"  Part="1"
+F 0 "C2" H 6125 1700 50  0000 L CNN
+F 1 "1u" H 6125 1500 50  0000 L CNN
+F 2 "Capacitors_SMD:C_0603" H 6138 1450 50  0001 C CNN
+F 3 "" H 6100 1600 50  0001 C CNN
+	1    6100 1600
+	1    0    0    -1
+$EndComp
+Wire Wire Line
+	6100 1300 6100 1450
+Connection ~ 6100 1300
+Wire Wire Line
+	6100 1750 6100 2950
+Connection ~ 6100 2950
 $EndSCHEMATC

Commit message: change to kicad 5
Parts:
- C1, C2: footprint Capacitors_SMD:C_0603 -> Capacitor_SMD:C_0603_1608Metric; symbol C -> Device:C
- Q1, Q2, Q3, Q5: footprint TO_SOT_Packages_SMD:SOT-23 -> Package_TO_SOT_SMD:SOT-23; symbol BC817 -> Transistor_BJT:BC817
- Q4, Q6: footprint TO_SOT_Packages_SMD:SOT-23 -> Package_TO_SOT_SMD:SOT-23; symbol BC807 -> Transistor_BJT:BC807
- Q7, Q8: symbol Q_NMOS_SGD -> Device:Q_NMOS_SGD
- R1, R2, R3, R4, R5, R6, R7: footprint Resistors_SMD:R_0603 -> Resistor_SMD:R_0603_1608Metric; symbol R -> Device:R

Commit message: smaller footprints
Parts:
- C1, C2: footprint Capacitor_SMD:C_0603_1608Metric -> _Generic:0603_Small
- Q1, Q2, Q3, Q4, Q5, Q6: footprint Package_TO_SOT_SMD:SOT-23 -> _Generic:SOT-23_Small
- Q7, Q8: footprint gmcontrol:DFN3x3A_8L_EP1_P -> _Generic:DFN3x3A_8L_EP1_P
- R1, R2, R3, R4, R5, R6, R7: footprint Resistor_SMD:R_0603_1608Metric -> _Generic:0603_Small
Changed lines of the file:
@@
 F 0 "Q5" H 7300 3825 50  0000 L CNN
 F 1 "BC817" H 7300 3750 50  0000 L CNN
-F 2 "Package_TO_SOT_SMD:SOT-23" H 7300 3675 50  0001 L CIN
+F 2 "_Generic:SOT-23_Small" H 7300 3675 50  0001 L CIN
 F 3 "" H 7100 3750 50  0001 L CNN
 	1    7100 3750
@@
 F 0 "Q2" H 6550 4425 50  0000 L CNN
 F 1 "BC817" H 6550 4350 50  0000 L CNN
-F 2 "Package_TO_SOT_SMD:SOT-23" H 6550 4275 50  0001 L CIN
+F 2 "_Generic:SOT-23_Small" H 6550 4275 50  0001 L CIN
 F 3 "" H 6350 4350 50  0001 L CNN
 	1    6350 4350
@@
 F 0 "Q6" H 7300 4425 50  0000 L CNN
 F 1 "BC807" H 7300 4350 50  0000 L CNN
-F 2 "Package_TO_SOT_SMD:SOT-23" H 7300 4275 50  0001 L CIN
+F 2 "_Generic:SOT-23_Small" H 7300 4275 50  0001 L CIN
 F 3 "" H 7100 4350 50  0001 L CNN
 	1    7100 4350
@@
 F 0 "R5" V 6530 3800 50  0000 C CNN
 F 1 "470" V 6450 3800 50  0000 C CNN
-F 2 "Resistor_SMD:R_0603_1608Metric" V 6380 3800 50  0001 C CNN
+F 2 "_Generic:0603_Small" V 6380 3800 50  0001 C CNN
 F 3 "" H 6450 3800 50  0001 C CNN
 	1    6450 3800
@@
 F 0 "R2" V 5880 4350 50  0000 C CNN
 F 1 "470" V 5800 4350 50  0000 C CNN
-F 2 "Resistor_SMD:R_0603_1608Metric" V 5730 4350 50  0001 C CNN
+F 2 "_Generic:0603_Small" V 5730 4350 50  0001 C CNN
 F 3 "" H 5800 4350 50  0001 C CNN
 	1    5800 4350
@@
 F 0 "Q8" H 7950 4100 50  0000 L CNN
 F 1 "AON7212" H 7950 4000 50  0000 L CNN
-F 2 "gmcontrol:DFN3x3A_8L_EP1_P" H 7950 4150 50  0001 C CNN
+F 2 "_Generic:DFN3x3A_8L_EP1_P" H 7950 4150 50  0001 C CNN
 F 3 "" H 7750 4050 50  0001 C CNN
 	1    7750 4050
@@
 F 0 "Q3" H 7300 1625 50  0000 L CNN
 F 1 "BC817" H 7300 1550 50  0000 L CNN
-F 2 "Package_TO_SOT_SMD:SOT-23" H 7300 1475 50  0001 L CIN
+F 2 "_Generic:SOT-23_Small" H 7300 1475 50  0001 L CIN
 F 3 "" H 7100 1550 50  0001 L CNN
 	1    7100 1550
@@
 F 0 "Q1" H 6550 2225 50  0000 L CNN
 F 1 "BC817" H 6550 2150 50  0000 L CNN
-F 2 "Package_TO_SOT_SMD:SOT-23" H 6550 2075 50  0001 L CIN
+F 2 "_Generic:SOT-23_Small" H 6550 2075 50  0001 L CIN
 F 3 "" H 6350 2150 50  0001 L CNN
 	1    6350 2150
@@
 F 0 "Q4" H 7300 2225 50  0000 L CNN
 F 1 "BC807" H 7300 2150 50  0000 L CNN
-F 2 "Package_TO_SOT_SMD:SOT-23" H 7300 2075 50  0001 L CIN
+F 2 "_Generic:SOT-23_Small" H 7300 2075 50  0001 L CIN
 F 3 "" H 7100 2150 50  0001 L CNN
 	1    7100 2150
@@
 F 0 "R3" V 6530 1600 50  0000 C CNN
 F 1 "470" V 6450 1600 50  0000 C CNN
-F 2 "Resistor_SMD:R_0603_1608Metric" V 6380 1600 50  0001 C CNN
+F 2 "_Generic:0603_Small" V 6380 1600 50  0001 C CNN
 F 3 "" H 6450 1600 50  0001 C CNN
 	1    6450 1600
@@
 F 0 "R1" V 5880 2150 50  0000 C CNN
 F 1 "470" V 5800 2150 50  0000 C CNN
-F 2 "Resistor_SMD:R_0603_1608Metric" V 5730 2150 50  0001 C CNN
+F 2 "_Generic:0603_Small" V 5730 2150 50  0001 C CNN
 F 3 "" H 5800 2150 50  0001 C CNN
 	1    5800 2150
@@
 F 0 "Q7" H 7950 1900 50  0000 L CNN
 F 1 "AON7212" H 7950 1800 50  0000 L CNN
-F 2 "gmcontrol:DFN3x3A_8L_EP1_P" H 7950 1950 50  0001 C CNN
+F 2 "_Generic:DFN3x3A_8L_EP1_P" H 7950 1950 50  0001 C CNN
 F 3 "" H 7750 1850 50  0001 C CNN
 	1    7750 1850
@@
 F 0 "R4" V 6530 2700 50  0000 C CNN
 F 1 "100" V 6450 2700 50  0000 C CNN
-F 2 "Resistor_SMD:R_0603_1608Metric" V 6380 2700 50  0001 C CNN
+F 2 "_Generic:0603_Small" V 6380 2700 50  0001 C CNN
 F 3 "" H 6450 2700 50  0001 C CNN
 	1    6450 2700
@@
 F 0 "R6" V 8830 3450 50  0000 C CNN
 F 1 "10k" V 8750 3450 50  0000 C CNN
-F 2 "Resistor_SMD:R_0603_1608Metric" V 8680 3450 50  0001 C CNN
+F 2 "_Generic:0603_Small" V 8680 3450 50  0001 C CNN
 F 3 "" H 8750 3450 50  0001 C CNN
 	1    8750 3450
@@
 F 0 "R7" V 8830 3950 50  0000 C CNN
 F 1 "1k" V 8750 3950 50  0000 C CNN
-F 2 "Resistor_SMD:R_0603_1608Metric" V 8680 3950 50  0001 C CNN
+F 2 "_Generic:0603_Small" V 8680 3950 50  0001 C CNN
 F 3 "" H 8750 3950 50  0001 C CNN
 	1    8750 3950
@@
 F 0 "C1" H 6075 3900 50  0000 L CNN
 F 1 "1u" H 6075 3700 50  0000 L CNN
-F 2 "Capacitor_SMD:C_0603_1608Metric" H 6088 3650 50  0001 C CNN
+F 2 "_Generic:0603_Small" H 6088 3650 50  0001 C CNN
 F 3 "" H 6050 3800 50  0001 C CNN
 	1    6050 3800
@@
 F 0 "C2" H 6125 1700 50  0000 L CNN
 F 1 "1u" H 6125 1500 50  0000 L CNN
-F 2 "Capacitor_SMD:C_0603_1608Metric" H 6138 1450 50  0001 C CNN
+F 2 "_Generic:0603_Small" H 6138 1450 50  0001 C CNN
 F 3 "" H 6100 1600 50  0001 C CNN
 	1    6100 1600

Commit message: basic layout
Changed lines of the file:
@@
 AR Path="/5AEA2A43/5AE6CAAE" Ref="Q21"  Part="1"
 AR Path="/5AEA319E/5AE6CAAE" Ref="Q29"  Part="1"
-F 0 "Q5" H 7300 3825 50  0000 L CNN
+F 0 "Q29" H 7300 3825 50  0000 L CNN
 F 1 "BC817" H 7300 3750 50  0000 L CNN
 F 2 "_Generic:SOT-23_Small" H 7300 3675 50  0001 L CIN
@@
 AR Path="/5AEA2A43/5AE6CB43" Ref="Q18"  Part="1"
 AR Path="/5AEA319E/5AE6CB43" Ref="Q26"  Part="1"
-F 0 "Q2" H 6550 4425 50  0000 L CNN
+F 0 "Q26" H 6550 4425 50  0000 L CNN
 F 1 "BC817" H 6550 4350 50  0000 L CNN
 F 2 "_Generic:SOT-23_Small" H 6550 4275 50  0001 L CIN
@@
 AR Path="/5AEA2A43/5AE6CB8C" Ref="Q22"  Part="1"
 AR Path="/5AEA319E/5AE6CB8C" Ref="Q30"  Part="1"
-F 0 "Q6" H 7300 4425 50  0000 L CNN
+F 0 "Q30" H 7300 4425 50  0000 L CNN
 F 1 "BC807" H 7300 4350 50  0000 L CNN
 F 2 "_Generic:SOT-23_Small" H 7300 4275 50  0001 L CIN
@@
 AR Path="/5AEA2A43/5AE6CC83" Ref="R22"  Part="1"
 AR Path="/5AEA319E/5AE6CC83" Ref="R29"  Part="1"
-F 0 "R5" V 6530 3800 50  0000 C CNN
+F 0 "R29" V 6530 3800 50  0000 C CNN
 F 1 "470" V 6450 3800 50  0000 C CNN
 F 2 "_Generic:0603_Small" V 6380 3800 50  0001 C CNN
@@
 AR Path="/5AEA2A43/5AE6CCF2" Ref="R19"  Part="1"
 AR Path="/5AEA319E/5AE6CCF2" Ref="R26"  Part="1"
-F 0 "R2" V 5880 4350 50  0000 C CNN
+F 0 "R26" V 5880 4350 50  0000 C CNN
 F 1 "470" V 5800 4350 50  0000 C CNN
 F 2 "_Generic:0603_Small" V 5730 4350 50  0001 C CNN
@@
 AR Path="/5AEA2A43/5AE6CEBE" Ref="Q24"  Part="1"
 AR Path="/5AEA319E/5AE6CEBE" Ref="Q32"  Part="1"
-F 0 "Q8" H 7950 4100 50  0000 L CNN
+F 0 "Q32" H 7950 4100 50  0000 L CNN
 F 1 "AON7212" H 7950 4000 50  0000 L CNN
 F 2 "_Generic:DFN3x3A_8L_EP1_P" H 7950 4150 50  0001 C CNN
@@
 AR Path="/5AEA2A43/5AE6DEA8" Ref="Q19"  Part="1"
 AR Path="/5AEA319E/5AE6DEA8" Ref="Q27"  Part="1"
-F 0 "Q3" H 7300 1625 50  0000 L CNN
+F 0 "Q27" H 7300 1625 50  0000 L CNN
 F 1 "BC817" H 7300 1550 50  0000 L CNN
 F 2 "_Generic:SOT-23_Small" H 7300 1475 50  0001 L CIN
@@
 AR Path="/5AEA2A43/5AE6DEAF" Ref="Q17"  Part="1"
 AR Path="/5AEA319E/5AE6DEAF" Ref="Q25"  Part="1"
-F 0 "Q1" H 6550 2225 50  0000 L CNN
+F 0 "Q25" H 6550 2225 50  0000 L CNN
 F 1 "BC817" H 6550 2150 50  0000 L CNN
 F 2 "_Generic:SOT-23_Small" H 6550 2075 50  0001 L CIN
@@
 AR Path="/5AEA2A43/5AE6DEB6" Ref="Q20"  Part="1"
 AR Path="/5AEA319E/5AE6DEB6" Ref="Q28"  Part="1"
-F 0 "Q4" H 7300 2225 50  0000 L CNN
+F 0 "Q28" H 7300 2225 50  0000 L CNN
 F 1 "BC807" H 7300 2150 50  0000 L CNN
 F 2 "_Generic:SOT-23_Small" H 7300 2075 50  0001 L CIN
@@
 AR Path="/5AEA2A43/5AE6DEBD" Ref="R20"  Part="1"
 AR Path="/5AEA319E/5AE6DEBD" Ref="R27"  Part="1"
-F 0 "R3" V 6530 1600 50  0000 C CNN
+F 0 "R27" V 6530 1600 50  0000 C CNN
 F 1 "470" V 6450 1600 50  0000 C CNN
 F 2 "_Generic:0603_Small" V 6380 1600 50  0001 C CNN
@@
 AR Path="/5AEA2A43/5AE6DEC4" Ref="R18"  Part="1"
 AR Path="/5AEA319E/5AE6DEC4" Ref="R25"  Part="1"
-F 0 "R1" V 5880 2150 50  0000 C CNN
+F 0 "R25" V 5880 2150 50  0000 C CNN
 F 1 "470" V 5800 2150 50  0000 C CNN
 F 2 "_Generic:0603_Small" V 5730 2150 50  0001 C CNN
@@
 AR Path="/5AEA2A43/5AE6DEDD" Ref="Q23"  Part="1"
 AR Path="/5AEA319E/5AE6DEDD" Ref="Q31"  Part="1"
-F 0 "Q7" H 7950 1900 50  0000 L CNN
+F 0 "Q31" H 7950 1900 50  0000 L CNN
 F 1 "AON7212" H 7950 1800 50  0000 L CNN
 F 2 "_Generic:DFN3x3A_8L_EP1_P" H 7950 1950 50  0001 C CNN
@@
 AR Path="/5AEA2A43/5AE6E0AE" Ref="R21"  Part="1"
 AR Path="/5AEA319E/5AE6E0AE" Ref="R28"  Part="1"
-F 0 "R4" V 6530 2700 50  0000 C CNN
+F 0 "R28" V 6530 2700 50  0000 C CNN
 F 1 "100" V 6450 2700 50  0000 C CNN
 F 2 "_Generic:0603_Small" V 6380 2700 50  0001 C CNN
@@
 AR Path="/5AEA2A43/5AE87A58" Ref="R23"  Part="1"
 AR Path="/5AEA319E/5AE87A58" Ref="R30"  Part="1"
-F 0 "R6" V 8830 3450 50  0000 C CNN
+F 0 "R30" V 8830 3450 50  0000 C CNN
 F 1 "10k" V 8750 3450 50  0000 C CNN
 F 2 "_Generic:0603_Small" V 8680 3450 50  0001 C CNN
@@
 AR Path="/5AEA2A43/5AE87B6A" Ref="R24"  Part="1"
 AR Path="/5AEA319E/5AE87B6A" Ref="R31"  Part="1"
-F 0 "R7" V 8830 3950 50  0000 C CNN
+F 0 "R31" V 8830 3950 50  0000 C CNN
 F 1 "1k" V 8750 3950 50  0000 C CNN
 F 2 "_Generic:0603_Small" V 8680 3950 50  0001 C CNN
@@
 AR Path="/5AEA2A43/5AE9E83C" Ref="C13"  Part="1"
 AR Path="/5AEA319E/5AE9E83C" Ref="C15"  Part="1"
-F 0 "C1" H 6075 3900 50  0000 L CNN
+F 0 "C15" H 6075 3900 50  0000 L CNN
 F 1 "1u" H 6075 3700 50  0000 L CNN
 F 2 "_Generic:0603_Small" H 6088 3650 50  0001 C CNN
@@
 AR Path="/5AEA2A43/5AE9EAA8" Ref="C14"  Part="1"
 AR Path="/5AEA319E/5AE9EAA8" Ref="C16"  Part="1"
-F 0 "C2" H 6125 1700 50  0000 L CNN
+F 0 "C16" H 6125 1700 50  0000 L CNN
 F 1 "1u" H 6125 1500 50  0000 L CNN
 F 2 "_Generic:0603_Small" H 6138 1450 50  0001 C CNN

Commit message: stm layout
Changed lines of the file:
@@
 AR Path="/5AEA2A43/5AE6CAAE" Ref="Q21"  Part="1"
 AR Path="/5AEA319E/5AE6CAAE" Ref="Q29"  Part="1"
-F 0 "Q29" H 7300 3825 50  0000 L CNN
+F 0 "Q5" H 7300 3825 50  0000 L CNN
 F 1 "BC817" H 7300 3750 50  0000 L CNN
 F 2 "_Generic:SOT-23_Small" H 7300 3675 50  0001 L CIN
@@
 AR Path="/5AEA2A43/5AE6CB43" Ref="Q18"  Part="1"
 AR Path="/5AEA319E/5AE6CB43" Ref="Q26"  Part="1"
-F 0 "Q26" H 6550 4425 50  0000 L CNN
+F 0 "Q2" H 6550 4425 50  0000 L CNN
 F 1 "BC817" H 6550 4350 50  0000 L CNN
 F 2 "_Generic:SOT-23_Small" H 6550 4275 50  0001 L CIN
@@
 AR Path="/5AEA2A43/5AE6CB8C" Ref="Q22"  Part="1"
 AR Path="/5AEA319E/5AE6CB8C" Ref="Q30"  Part="1"
-F 0 "Q30" H 7300 4425 50  0000 L CNN
+F 0 "Q6" H 7300 4425 50  0000 L CNN
 F 1 "BC807" H 7300 4350 50  0000 L CNN
 F 2 "_Generic:SOT-23_Small" H 7300 4275 50  0001 L CIN
@@
 AR Path="/5AEA2A43/5AE6CC83" Ref="R22"  Part="1"
 AR Path="/5AEA319E/5AE6CC83" Ref="R29"  Part="1"
-F 0 "R29" V 6530 3800 50  0000 C CNN
+F 0 "R5" V 6530 3800 50  0000 C CNN
 F 1 "470" V 6450 3800 50  0000 C CNN
 F 2 "_Generic:0603_Small" V 6380 3800 50  0001 C CNN
@@
 AR Path="/5AEA2A43/5AE6CCF2" Ref="R19"  Part="1"
 AR Path="/5AEA319E/5AE6CCF2" Ref="R26"  Part="1"
-F 0 "R26" V 5880 4350 50  0000 C CNN
+F 0 "R2" V 5880 4350 50  0000 C CNN
 F 1 "470" V 5800 4350 50  0000 C CNN
 F 2 "_Generic:0603_Small" V 5730 4350 50  0001 C CNN
@@
 AR Path="/5AEA2A43/5AE6CEBE" Ref="Q24"  Part="1"
 AR Path="/5AEA319E/5AE6CEBE" Ref="Q32"  Part="1"
-F 0 "Q32" H 7950 4100 50  0000 L CNN
+F 0 "Q8" H 7950 4100 50  0000 L CNN
 F 1 "AON7212" H 7950 4000 50  0000 L CNN
 F 2 "_Generic:DFN3x3A_8L_EP1_P" H 7950 4150 50  0001 C CNN
@@
 AR Path="/5AEA2A43/5AE6DEA8" Ref="Q19"  Part="1"
 AR Path="/5AEA319E/5AE6DEA8" Ref="Q27"  Part="1"
-F 0 "Q27" H 7300 1625 50  0000 L CNN
+F 0 "Q3" H 7300 1625 50  0000 L CNN
 F 1 "BC817" H 7300 1550 50  0000 L CNN
 F 2 "_Generic:SOT-23_Small" H 7300 1475 50  0001 L CIN
@@
 AR Path="/5AEA2A43/5AE6DEAF" Ref="Q17"  Part="1"
 AR Path="/5AEA319E/5AE6DEAF" Ref="Q25"  Part="1"
-F 0 "Q25" H 6550 2225 50  0000 L CNN
+F 0 "Q1" H 6550 2225 50  0000 L CNN
 F 1 "BC817" H 6550 2150 50  0000 L CNN
 F 2 "_Generic:SOT-23_Small" H 6550 2075 50  0001 L CIN
@@
 AR Path="/5AEA2A43/5AE6DEB6" Ref="Q20"  Part="1"
 AR Path="/5AEA319E/5AE6DEB6" Ref="Q28"  Part="1"
-F 0 "Q28" H 7300 2225 50  0000 L CNN
+F 0 "Q4" H 7300 2225 50  0000 L CNN
 F 1 "BC807" H 7300 2150 50  0000 L CNN
 F 2 "_Generic:SOT-23_Small" H 7300 2075 50  0001 L CIN
@@
 AR Path="/5AEA2A43/5AE6DEBD" Ref="R20"  Part="1"
 AR Path="/5AEA319E/5AE6DEBD" Ref="R27"  Part="1"
-F 0 "R27" V 6530 1600 50  0000 C CNN
+F 0 "R3" V 6530 1600 50  0000 C CNN
 F 1 "470" V 6450 1600 50  0000 C CNN
 F 2 "_Generic:0603_Small" V 6380 1600 50  0001 C CNN
@@
 AR Path="/5AEA2A43/5AE6DEC4" Ref="R18"  Part="1"
 AR Path="/5AEA319E/5AE6DEC4" Ref="R25"  Part="1"
-F 0 "R25" V 5880 2150 50  0000 C CNN
+F 0 "R1" V 5880 2150 50  0000 C CNN
 F 1 "470" V 5800 2150 50  0000 C CNN
 F 2 "_Generic:0603_Small" V 5730 2150 50  0001 C CNN
@@
 AR Path="/5AEA2A43/5AE6DEDD" Ref="Q23"  Part="1"
 AR Path="/5AEA319E/5AE6DEDD" Ref="Q31"  Part="1"
-F 0 "Q31" H 7950 1900 50  0000 L CNN
+F 0 "Q7" H 7950 1900 50  0000 L CNN
 F 1 "AON7212" H 7950 1800 50  0000 L CNN
 F 2 "_Generic:DFN3x3A_8L_EP1_P" H 7950 1950 50  0001 C CNN
@@
 AR Path="/5AEA2A43/5AE6E0AE" Ref="R21"  Part="1"
 AR Path="/5AEA319E/5AE6E0AE" Ref="R28"  Part="1"
-F 0 "R28" V 6530 2700 50  0000 C CNN
+F 0 "R4" V 6530 2700 50  0000 C CNN
 F 1 "100" V 6450 2700 50  0000 C CNN
 F 2 "_Generic:0603_Small" V 6380 2700 50  0001 C CNN
@@
 AR Path="/5AEA2A43/5AE87A58" Ref="R23"  Part="1"
 AR Path="/5AEA319E/5AE87A58" Ref="R30"  Part="1"
-F 0 "R30" V 8830 3450 50  0000 C CNN
+F 0 "R6" V 8830 3450 50  0000 C CNN
 F 1 "10k" V 8750 3450 50  0000 C CNN
 F 2 "_Generic:0603_Small" V 8680 3450 50  0001 C CNN
@@
 AR Path="/5AEA2A43/5AE87B6A" Ref="R24"  Part="1"
 AR Path="/5AEA319E/5AE87B6A" Ref="R31"  Part="1"
-F 0 "R31" V 8830 3950 50  0000 C CNN
+F 0 "R7" V 8830 3950 50  0000 C CNN
 F 1 "1k" V 8750 3950 50  0000 C CNN
 F 2 "_Generic:0603_Small" V 8680 3950 50  0001 C CNN
@@
 AR Path="/5AEA2A43/5AE9E83C" Ref="C13"  Part="1"
 AR Path="/5AEA319E/5AE9E83C" Ref="C15"  Part="1"
-F 0 "C15" H 6075 3900 50  0000 L CNN
+F 0 "C1" H 6075 3900 50  0000 L CNN
 F 1 "1u" H 6075 3700 50  0000 L CNN
 F 2 "_Generic:0603_Small" H 6088 3650 50  0001 C CNN
@@
 AR Path="/5AEA2A43/5AE9EAA8" Ref="C14"  Part="1"
 AR Path="/5AEA319E/5AE9EAA8" Ref="C16"  Part="1"
-F 0 "C16" H 6125 1700 50  0000 L CNN
+F 0 "C2" H 6125 1700 50  0000 L CNN
 F 1 "1u" H 6125 1500 50  0000 L CNN
 F 2 "_Generic:0603_Small" H 6138 1450 50  0001 C CNN
