File: hardware/gmcontrol.kicad_pcb (KiCad board)
At the start: 2 copper layers, 114 parts, among them J1 USB_OTG, J2 Jack-DC, Q1 BC817, Q10 BC817, Q11 BC817, Q12 BC807, Q13 BC817, Q14 BC807, Q15 AON7212, Q16 AON7212, Q17 BC817, Q18 BC817, Q19 BC817, Q2 BC817, Q20 BC807, Q21 BC817, Q22 BC807, Q23 AON7212, Q24 AON7212, Q25 BC817, Q26 BC817, Q27 BC817, Q28 BC807, Q29 BC817, Q3 BC817, Q30 BC807, Q31 AON7212, Q32 AON7212, Q33 BSS138, Q34 BC817, Q35 BSS84, Q36 AO3401, Q4 BC807, Q5 BC817, Q6 BC807, Q7 AON7212, Q8 AON7212, Q9 BC817, U1 STM32F103C8Tx, U2 HT7333-1, Y1 16Mhz

Commit message: multiple phases
Parts:
- C22, Q1, Q10, Q12, Q14, Q2, Q25, Q26, Q28, Q30, Q4, Q6, Q9, R16, R30, R6: moved to B.Cu
- moved R6 88.8 mm to (145.1, 39.3), turned to 90 degrees
- moved C12 88.0 mm to (155.4, 42.6), turned to 270 degrees
- moved R15 87.1 mm to (150.7, 43.1), turned to 270 degrees
- moved Q15 86.9 mm to (154.3, 38.1)
- moved R5 85.1 mm to (143.5, 43.1), turned to 270 degrees
- moved C11 83.4 mm to (149.6, 43.1), turned to 270 degrees
- moved R17 82.9 mm to (151.9, 43.1), turned to 90 degrees
- moved R4 82.5 mm to (145.3, 44.7), turned to 180 degrees
- moved R2 81.9 mm to (143.0, 44.7), turned to 180 degrees
- moved R11 81.6 mm to (154.8, 44.3), turned to 180 degrees
- moved R7 81.1 mm to (144.6, 43.1), turned to 90 degrees
- moved R3 80.3 mm to (146.1, 42.6), turned to 90 degrees
- moved R13 79.4 mm to (153.3, 42.6), turned to 90 degrees
- moved R30 79.2 mm to (159.6, 39.3), turned to 90 degrees
- moved Q16 78.9 mm to (150.7, 38.1)
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Routing:
- net /controller/GND: track 20.0 -> 94.5 mm, vias 7 -> 28
- net /gate_voltage_supply/Vgl: track 3.17 -> 36.7 mm, vias 1 -> 4
- net /gate_voltage_supply/Vgh: track 5.77 -> 38.1 mm, vias 1 -> 4
- net /gate_voltage_supply/VIN: track 10.7 -> 37.4 mm, vias 0 -> 56
- net /sheet5AEA1DE6/PHASE: track 0.00 -> 17.0 mm, vias 0 -> 16
- net /phase_driver_1/PHASE: track 0.00 -> 17.0 mm, vias 0 -> 16
- net /sheet5AEA3194/PHASE: track 0.00 -> 17.0 mm, vias 0 -> 16
- net /sheet5AEA2A39/PHASE: track 10.1 -> 17.0 mm, vias 1 -> 16
- net /sheet5AEA3194/SENSE: track 0.00 -> 5.98 mm, vias 0 -> 1
- net /sheet5AEA1DE6/SENSE: track 0.00 -> 5.98 mm, vias 0 -> 1
- net /phase_driver_1/SENSE: track 0.00 -> 5.98 mm, vias 0 -> 1
- net Net-(Q10-Pad3): track 0.00 -> 5.38 mm, vias 0 -> 2
- net Net-(Q26-Pad3): track 0.00 -> 5.38 mm, vias 0 -> 2
- net Net-(Q2-Pad3): track 0.00 -> 5.38 mm, vias 0 -> 2
- net Net-(Q1-Pad3): track 0.00 -> 5.04 mm, vias 0 -> 1
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- added copper zone on F.Cu, net /controller/GND
- added copper zone on B.Cu, net /gate_voltage_supply/VIN
- added copper zone on B.Cu, net /phase_driver_1/PHASE
- added copper zone on F.Cu, net /phase_driver_1/PHASE
- added copper zone on B.Cu, net /sheet5AEA1DE6/PHASE
- added copper zone on F.Cu, net /sheet5AEA1DE6/PHASE
- added copper zone on B.Cu, net /sheet5AEA2A39/PHASE
- added copper zone on F.Cu, net /sheet5AEA2A39/PHASE
- added copper zone on B.Cu, net /sheet5AEA3194/PHASE
- added copper zone on F.Cu, net /sheet5AEA3194/PHASE
- added copper zone on F.Cu, net Net-(Q11-Pad2)
- added copper zone on F.Cu, net Net-(Q13-Pad2)
- added copper zone on F.Cu, net Net-(Q19-Pad2)
- added copper zone on F.Cu, net Net-(Q27-Pad2)
- added copper zone on F.Cu, net Net-(Q29-Pad2)
- added copper zone on F.Cu, net Net-(Q3-Pad2)
- added copper zone on F.Cu, net Net-(Q5-Pad2)
- removed copper zone on B.Cu, net /controller/GND

Commit message: power layout
Parts:
- added C25: 22u, _Generic:0805_Small, B.Cu at (156.2, 36.1)
- added C26: 22u, _Generic:0805_Small, B.Cu at (156.2, 37.4)
- added C27: 22u, _Generic:0805_Small, B.Cu at (134.5, 37.4)
- added C28: 22u, _Generic:0805_Small, B.Cu at (134.5, 36.1)
- J1: moved to B.Cu
- moved J2 113.7 mm to (128.5, 41.6), turned to 90 degrees
- moved J1 109.2 mm to (128.7, 53.3), turned to 180 degrees
- moved Q36 91.5 mm to (135.4, 49.8), turned to 180 degrees
- moved U2 81.5 mm to (140.5, 53.8), turned to 270 degrees
- moved C24 72.3 mm to (151.6, 59.9)
- moved R43 72.3 mm to (155.1, 59.9)
- moved R41 71.0 mm to (144.3, 71.4)
- moved C20 71.0 mm to (144.8, 66.4)
- moved R42 71.0 mm to (148.6, 66.4)
- moved U1 68.6 mm to (153.9, 53.0)
- moved R8 65.1 mm to (163.5, 63.5)
- moved C4 65.1 mm to (168.8, 56.5)
- moved C6 65.1 mm to (167.7, 61.5)
- moved R10 65.1 mm to (163.7, 58.5)
- moved R9 65.1 mm to (168.8, 51.6)
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Routing:
- net /gate_voltage_supply/VIN: track 37.4 -> 82.1 mm
- net /gate_voltage_supply/Vgl: track 36.7 -> 71.6 mm, vias 4 -> 12
- net /gate_voltage_supply/Vgh: track 38.1 -> 70.7 mm, vias 4 -> 13
- net /sheet5AEA2A39/PHASE: track 17.0 -> 17.5 mm, vias 16 -> 15
- net /sheet5AEA1DE6/PHASE: vias 16 -> 15
- net /phase_driver_1/PHASE: vias 16 -> 15
- added copper zone on B.Cu, net /controller/GND
Other:
- board outline added: 40 x 25 mm

Commit message: basic layout
Parts:
- added C29: 22u, _Generic:0805_Small, B.Cu at (158.1, 33.9)
- added C30: 22u, _Generic:0805_Small, B.Cu at (159.5, 33.9)
- C10, C9, D4, Q33, Q34, Q35, Q36, R33, R36, R41, R8, R9: moved to B.Cu
- moved C10 44.8 mm to (132.4, 50.6)
- moved C9 43.8 mm to (132.6, 51.8), turned to 180 degrees
- moved R9 36.5 mm to (132.5, 48.3), turned to 180 degrees
- moved R8 34.1 mm to (132.4, 49.4), turned to 180 degrees
- moved L2 32.9 mm to (132.7, 36.5)
- moved R41 29.1 mm to (130.8, 45.6), turned to 90 degrees
- moved C3 27.8 mm to (144.2, 55.9)
- moved R10 27.8 mm to (136.5, 52.8)
- moved C4 27.4 mm to (141.8, 52.2)
- moved L1 25.2 mm to (126.4, 39.2), turned to 180 degrees
- moved Q35 25.0 mm to (131.5, 36.6)
- moved C5 24.5 mm to (148.9, 50.2)
- moved Q34 24.0 mm to (132.1, 39.9), turned to 90 degrees
- moved Y1 23.4 mm to (141.2, 54.9)
- moved Q33 23.2 mm to (125.9, 39.3), turned to 180 degrees
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Routing:
- net /gate_voltage_supply/VIN: track 82.1 -> 69.1 mm
- net /gate_voltage_supply/Vgl: track 71.6 -> 68.6 mm, vias 12 -> 11

Commit message: stm layout
Parts:
- added J3: Conn_01x18, Connector_PinSocket_2.54mm:PinSocket_1x18_P2.54mm_Horizontal, F.Cu at (204.8, 38.1)
- added J4: Screw_Terminal_01x04, TerminalBlock:TerminalBlock_bornier-4_P5.08mm, F.Cu at (141.1, 15.8)
- added REF**: MountingHole_2.2mm_M2_ISO7380_Pad, MountingHole:MountingHole_2.2mm_M2_ISO7380_Pad, F.Cu at (136.0, 55.0)
- added REF**: MountingHole_2.2mm_M2_ISO7380_Pad, MountingHole:MountingHole_2.2mm_M2_ISO7380_Pad, F.Cu at (162.0, 55.0)
- C17, C20, C24, C3, C4, C5, C6, C7, C8, D3, R10, R34, R35: moved to B.Cu
- J2: footprint Connector_BarrelJack:BarrelJack_Horizontal -> gmcontrol:BarrelJack_Horizontal_modified
- moved C7 11.0 mm to (145.9, 53.9)
- moved C24 8.71 mm to (139.9, 49.4), turned to 270 degrees
- moved C8 7.10 mm to (143.5, 53.6), turned to 90 degrees
- moved C5 5.13 mm to (144.5, 47.5)
- moved C6 4.93 mm to (150.1, 48.1), turned to 270 degrees
- moved D3 4.70 mm to (125.5, 35.6), turned to 90 degrees
- moved R43 4.39 mm to (137.8, 46.9), turned to 270 degrees
- moved C20 4.21 mm to (138.8, 49.4), turned to 90 degrees
- moved C3 3.72 mm to (140.8, 54.4), turned to 90 degrees
- moved C4 3.46 mm to (139.1, 54.4), turned to 270 degrees
- moved R32 3.26 mm to (128.2, 36.8), turned to 0 degrees
- moved C9 3.18 mm to (131.7, 48.7), turned to 0 degrees
- moved R42 2.87 mm to (138.9, 46.9), turned to 270 degrees
- moved R10 2.81 mm to (134.3, 51.0)
- moved R35 2.74 mm to (132.5, 37.5)
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Connections:
- U1 pad 17: (no net) -> /controller/PA7
- U1 pad 18: (no net) -> /controller/PB0
- U1 pad 19: (no net) -> /controller/PB1
- U1 pad 2: (no net) -> /controller/PC13
- U1 pad 20: (no net) -> /controller/PB2
- U1 pad 25: (no net) -> /controller/PB12
- U1 pad 3: (no net) -> /controller/PC14
- U1 pad 34: (no net) -> /controller/SWDIO
- U1 pad 37: (no net) -> /controller/SWDCLK
- U1 pad 38: (no net) -> /controller/PA15
- U1 pad 39: (no net) -> /controller/PB3
- U1 pad 4: (no net) -> /controller/PC15
- U1 pad 40: (no net) -> /controller/PB4
- U1 pad 41: (no net) -> /controller/PB5
- U1 pad 42: (no net) -> /controller/PB6
- U1 pad 43: (no net) -> /controller/PB7
- U1 pad 44: (no net) -> /controller/BOOT0
- U1 pad 5: Net-(U1-Pad5) -> Net-(C3-Pad1)
- U1 pad 6: Net-(U1-Pad6) -> Net-(C4-Pad1)
- U1 pad 7: (no net) -> /controller/RESET
- Y1 pad 1: Net-(U1-Pad5) -> Net-(C3-Pad1)
- Y1 pad 2: Net-(C3-Pad1) -> /controller/GND
- Y1 pad 3: Net-(U1-Pad6) -> Net-(C4-Pad1)
- Y1 pad 4: Net-(C4-Pad1) -> /controller/GND
Routing:
- net /controller/GND: track 94.5 -> 219.6 mm, vias 28 -> 35
- net /gate_voltage_supply/VIN: track 69.1 -> 136.0 mm, vias 56 -> 58
- net /power/3.3V: track 0.00 -> 45.8 mm, vias 0 -> 7
- net /controller/SENSE_Vgh: track 0.00 -> 33.5 mm, vias 0 -> 2
- net /controller/SENSE_Vgl: track 0.00 -> 24.2 mm, vias 0 -> 2
- net /controller/CLK_Vgh: track 0.00 -> 23.7 mm
- net /sheet5AEA2A39/SENSE: track 5.98 -> 25.7 mm, vias 1 -> 3
- net Net-(R8-Pad1): track 0.00 -> 17.7 mm, vias 0 -> 3
- net /controller/CLK_Vgl: track 0.00 -> 17.5 mm, vias 0 -> 1
- net /controller/SENSE_Vmotor: track 0.00 -> 17.3 mm, vias 0 -> 2
- net /sheet5AEA3194/SENSE: track 5.98 -> 22.9 mm, vias 1 -> 3
- net /phase_driver_1/SENSE: track 5.98 -> 22.6 mm
- net /gate_voltage_supply/Vgh: track 70.7 -> 86.3 mm, vias 13 -> 15
- net Net-(R9-Pad1): track 0.00 -> 15.3 mm, vias 0 -> 3
- net /controller/PA15: track 0.00 -> 13.8 mm, vias 0 -> 2
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Other:
- outline, holes or cut-outs redrawn

Commit message: vin
Parts:
- moved R41 0.61 mm to (130.9, 46.2), turned to 270 degrees
- moved Q36 0.45 mm to (128.7, 46.2)
Routing:
- net /power/Vusb: track 6.34 -> 17.3 mm, vias 2 -> 8
- net /gate_voltage_supply/VIN: track 136.0 -> 141.1 mm, vias 58 -> 59
- net /controller/GND: track 219.6 -> 220.1 mm
- net /power/3.3V: track 45.8 -> 46.3 mm
- added copper zone on B.Cu, net /power/Vusb
