File: hardware/gmcontrol.kicad_pcb (KiCad board)
At the start: 2 copper layers, 40 x 25 mm, 124 parts, among them J1 USB_OTG, J2 Jack-DC, J3 Conn_01x18, J4 Screw_Terminal_01x04, Q1 BC817, Q10 BC817, Q11 BC817, Q12 BC807, Q13 BC817, Q14 BC807, Q15 AON7212, Q16 AON7212, Q17 BC817, Q18 BC817, Q19 BC817, Q2 BC817, Q20 BC807, Q21 BC817, Q22 BC807, Q23 AON7212, Q24 AON7212, Q25 BC817, Q26 BC817, Q27 BC817, Q28 BC807, Q29 BC817, Q3 BC817, Q30 BC807, Q31 AON7212, Q32 AON7212, Q33 BSS138, Q34 BC817, Q35 BSS84, Q36 AO3401, Q4 BC807, Q5 BC817, Q6 BC807, Q7 AON7212, Q8 AON7212, Q9 BC817, U1 STM32F103C8Tx, U2 HT7333-1, Y1 16Mhz

Commit message: finished pcb design
Parts:
- removed J4: Screw_Terminal_01x04, TerminalBlock:TerminalBlock_bornier-4_P5.08mm
- removed REF** (x2): MountingHole_2.2mm_M2_ISO7380_Pad, MountingHole:MountingHole_2.2mm_M2_ISO7380_Pad
- added J10: Conn_01x01, _Generic:2.54Pad, F.Cu at (162.6, 52.7)
- added J11: Conn_01x01, _Generic:1.27Pad, F.Cu at (156.2, 46.9)
- added J12: Conn_01x01, _Generic:1.27Pad, F.Cu at (150.9, 55.3)
- added J13: Conn_01x01, _Generic:1.27Pad, F.Cu at (157.5, 48.1)
- added J14: Conn_01x01, _Generic:1.27Pad, F.Cu at (158.8, 48.1)
- added J15: Conn_01x01, _Generic:1.27Pad, F.Cu at (160.0, 46.9)
- added J16: Conn_01x01, _Generic:1.27Pad, F.Cu at (161.3, 46.9)
- added J17: Conn_01x01, _Generic:1.27Pad, F.Cu at (162.6, 46.9)
- added J18: Conn_01x01, _Generic:1.27Pad, F.Cu at (160.0, 48.1)
- added J19: Conn_01x01, _Generic:1.27Pad, F.Cu at (161.3, 48.1)
- added J20: Conn_01x01, _Generic:1.27Pad, F.Cu at (162.6, 48.1)
- added J21: Conn_01x01, _Generic:1.27Pad, F.Cu at (158.8, 46.9)
- added J22: Conn_01x01, _Generic:1.27Pad, F.Cu at (156.8, 55.9)
- added J23: Conn_01x01, _Generic:1.27Pad, F.Cu at (158.1, 55.9)
- added J24: Conn_01x01, _Generic:1.27Pad, F.Cu at (159.4, 55.9)
- added J25: Conn_01x01, _Generic:1.27Pad, F.Cu at (137.7, 53.2)
- added J26: Conn_01x01, _Generic:1.27Pad, F.Cu at (157.5, 46.9)
- added J5: Conn_01x01, _Generic:2.54Pad, F.Cu at (160.0, 50.2)
- added J6: Conn_01x01, _Generic:2.54Pad, F.Cu at (157.5, 50.2)
- added J7: Conn_01x01, _Generic:2.54Pad, F.Cu at (162.6, 50.2)
- added J8: Conn_01x01, _Generic:2.54Pad, F.Cu at (157.5, 52.7)
- added J9: Conn_01x01, _Generic:2.54Pad, F.Cu at (160.0, 52.7)
- added MK1: Mounting_Hole_PAD, MountingHole:MountingHole_2.2mm_M2_ISO7380_Pad, F.Cu at (136.0, 55.0)
- added MK2: Mounting_Hole_PAD, MountingHole:MountingHole_2.2mm_M2_ISO7380_Pad, F.Cu at (162.0, 55.0)
- J3: value Conn_01x18 -> Conn_01x01; footprint Connector_PinSocket_2.54mm:PinSocket_1x18_P2.54mm_Horizontal -> _Generic:1.27Pad
- moved J3 49.6 mm to (156.2, 48.1)
- moved C6 1.37 mm to (151.5, 47.9)
- moved R12 0.27 mm to (149.7, 44.2)
- moved R4 0.06 mm to (145.7, 43.5)
- moved R21 0.05 mm to (138.5, 43.5)
- moved R11 0.05 mm to (155.3, 43.0)
- moved R19 0.05 mm to (136.7, 44.3)
Connections:
- J3 pad 1: /controller/SWDIO -> /controller/GND
Routing:
- net /controller/GND: track 220.1 -> 264.2 mm, vias 35 -> 51
- net /gate_voltage_supply/Vgh: track 86.3 -> 100.4 mm
- net /controller/PB5: track 12.4 -> 25.7 mm
- net /controller/RESET: track 6.74 -> 19.5 mm
- net /controller/PB2: track 3.03 -> 14.9 mm
- net /controller/PB4: track 13.1 -> 24.9 mm
- net /controller/SWDIO: track 10.1 -> 20.5 mm, vias 2 -> 4
- net /controller/PB1: track 3.21 -> 13.5 mm
- net /power/3.3V: track 46.3 -> 56.4 mm, vias 7 -> 9
- net /controller/PB7: track 11.0 -> 20.5 mm
- net /controller/PB0: track 3.39 -> 12.1 mm
- net /controller/PB3: track 13.6 -> 22.2 mm
- net /gate_voltage_supply/Vgl: track 72.6 -> 79.8 mm
- net /controller/SWDCLK: track 13.6 -> 20.8 mm
- net /controller/PB12: track 4.11 -> 11.2 mm, vias 2 -> 3
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- added copper zone on F.Cu, net /gate_voltage_supply/VIN
- added copper zone on F.Cu, net /power/3.3V
- added copper zone on F.Cu, net /power/Vusb
Other:
- net class 3.3V added: clearance 0.15, trace_width 0.2, via_dia 0.6, via_drill 0.4
- net class VIN added: clearance 0.15, trace_width 0.5, via_dia 0.6, via_drill 0.4
- rule trace_min: 0.127 -> 0.15
