File: hardware/gmcontrol.kicad_pcb (KiCad board)
At the start: 2 copper layers, 40 x 25 mm, 145 parts, among them J1 USB_OTG, J10 Conn_01x01, J11 Conn_01x01, J12 Conn_01x01, J13 Conn_01x01, J14 Conn_01x01, J15 Conn_01x01, J16 Conn_01x01, J17 Conn_01x01, J18 Conn_01x01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

Commit message: Ordered V1 PCB version
Parts:
- R36: value 200 -> 220
- moved J12 0.72 mm to (150.9, 54.5)
Routing:
- net /controller/BOOT0: track 10.5 -> 9.99 mm, vias 2 -> 1
